File: hardware/0.1/pro-micro-c.kicad_pcb (KiCad board)
At the start: 2 copper layers, 20.4 x 34.3 mm, 24 parts, among them J1 USB_C_Receptacle_USB2.0, J2 0.1" x 12, J3 0.1" x 5, J4 0.1" x 12, SW1 SW_Push, U1 USBLC6-2P6, U2 ATmega32U4-MU, Y1 16MHz

Commit message: v0.2
Parts:
- added G***: LOGO, josh-logos:OSHW_Logo_3.6x3.6_F.Mask, B.Cu at (186.5, 79.4)
- added G***: LOGO, josh-logos:josh-johnson-logo-8_6x1_5, B.Cu at (184.9, 66.0)
- added REF**: Josh Details, josh-logos:josh-details, B.Cu at (186.0, 66.5)
Routing:
- net /nRST: track 27.2 -> 27.9 mm
- net GND: track 72.6 -> 73.1 mm, vias 28 -> 20
- net (no net): vias 4 -> 0
