File: hardware/0.2/pro-micro-c.kicad_pcb (KiCad board)
At the start: 2 copper layers, 20.4 x 34.3 mm, 27 parts, among them J1 USB_C_Receptacle_USB2.0, J2 0.1" x 12, J3 0.1" x 5, J4 0.1" x 12, SW1 SW_Push, U1 USBLC6-2P6, U2 ATmega32U4-MU, Y1 16MHz

Commit message: update files + readme
Parts:
- removed the G*** at (181.0, 62.5)
- J2, J4: footprint josh-connectors:Castellated_P2.54x12 -> josh-connectors:Castellated_Short_P2.54x12
- J3: footprint josh-connectors:Castellated_P2.54x5 -> josh-connectors:Castellated_Short_2.54x5
- moved REF** 0.10 mm to (182.1, 63.1)
Routing:
- net GND: track 84.3 -> 75.7 mm
- net /PB6: track 17.6 -> 15.4 mm
- net /PF7: track 6.74 -> 4.49 mm
- net /PB3: track 21.5 -> 19.3 mm
- net /PB2: track 23.1 -> 20.9 mm
- net /PB1: track 19.8 -> 17.5 mm
- net /PF1: track 15.9 -> 13.6 mm
- net /PF0: track 16.7 -> 14.4 mm
- net /PD5: track 18.5 -> 16.2 mm
- net /PC7: track 10.8 -> 8.62 mm
- net /PB7: track 28.8 -> 26.6 mm
- net /PE6: track 35.7 -> 33.5 mm
- net /PD7: track 11.9 -> 9.72 mm
- net /PC6: track 15.0 -> 12.8 mm
- net /PB5: track 16.3 -> 14.1 mm
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Other:
- board size 20.4 x 34.3 mm -> 18 x 33.1 mm
- board text added: "G"
- board text added: "VB"
- board text removed: "VBUS"
