File: hardware/0.2/pro-micro-c.sch (KiCad schematic (older format))
At the start: 24 parts, among them J1 USB_C_Receptacle_USB2.0, J2 0.1\" x 12, J3 0.1\" x 5, J4 0.1\" x 12, SW1 SW_Push, U1 USBLC6-2P6, U2 ATmega32U4-MU, Y1 16MHz

Commit message: update files + readme
Parts:
- J2, J4: footprint josh-connectors:Castellated_P2.54x12 -> josh-connectors:Castellated_Short_P2.54x12
- J3: footprint josh-connectors:Castellated_P2.54x5 -> josh-connectors:Castellated_Short_2.54x5
Changed lines of the file:
@@
 F 0 "J3" V 3212 5644 50  0000 L CNN
 F 1 "0.1\" x 5" V 3303 5644 50  0000 L CNN
-F 2 "josh-connectors:Castellated_P2.54x5" H 3150 5400 50  0001 C CNN
+F 2 "josh-connectors:Castellated_Short_2.54x5" H 3150 5400 50  0001 C CNN
 F 3 "~" H 3150 5400 50  0001 C CNN
 	1    3150 5400
@@
 F 0 "J2" H 3100 4000 50  0000 R CNN
 F 1 "0.1\" x 12" H 3100 4100 50  0000 R CNN
-F 2 "josh-connectors:Castellated_P2.54x12" H 2900 4850 50  0001 C CNN
+F 2 "josh-connectors:Castellated_Short_P2.54x12" H 2900 4850 50  0001 C CNN
 F 3 "~" H 2900 4850 50  0001 C CNN
 	1    2900 4850
@@
 F 0 "J4" H 3350 5500 50  0000 C CNN
 F 1 "0.1\" x 12" H 3500 5400 50  0000 C CNN
-F 2 "josh-connectors:Castellated_P2.54x12" H 3400 4750 50  0001 C CNN
+F 2 "josh-connectors:Castellated_Short_P2.54x12" H 3400 4750 50  0001 C CNN
 F 3 "~" H 3400 4750 50  0001 C CNN
 	1    3400 4750
