File: hardware/0.3/pro-micro-c.kicad_pcb (KiCad board)
At the start: 2 copper layers, 18 x 33.1 mm, 22 parts, among them J1 USB_C_Receptacle_USB2.0, J2 0.1" x 12, J3 0.1" x 12, U1 ATmega32U4-MU, Y1 16MHz

Commit message: layout looking good
Parts:
- added SW1: KMR2, josh-buttons-switches:SW_Push_KMR2, F.Cu at (146.8, 94.4)
- D1: footprint Diode_SMD:D_SOD-123F -> josh-passives-smt:D_SOD-123F
- moved J3 77.9 mm to (121.1, 91.3), turned to 90 degrees
- moved J1 73.5 mm to (122.6, 98.9), turned to 270 degrees
- moved R4 67.7 mm to (128.3, 93.1), turned to 180 degrees
- moved F1 67.1 mm to (128.3, 94.7), turned to 180 degrees
- moved R1 66.5 mm to (128.3, 96.2), turned to 180 degrees
- moved R6 66.0 mm to (128.3, 97.7), turned to 180 degrees
- moved R5 65.6 mm to (128.3, 99.2), turned to 180 degrees
- moved R2 65.2 mm to (128.3, 100.7), turned to 180 degrees
- moved R3 64.8 mm to (128.3, 102.5), turned to 180 degrees
- moved D2 64.6 mm to (128.3, 104.1), turned to 180 degrees
- moved D1 63.5 mm to (131.0, 94.9), turned to 270 degrees
- moved C4 60.1 mm to (132.1, 98.8), turned to 180 degrees
- moved C5 59.6 mm to (132.1, 100.3), turned to 0 degrees
- moved C6 57.3 mm to (133.2, 104.0), turned to 180 degrees
- moved C3 57.0 mm to (135.8, 94.0), turned to 180 degrees
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Routing:
- net /nRST: track 20.6 -> 43.0 mm, vias 0 -> 2
- net GND: track 38.6 -> 51.9 mm, vias 15 -> 23
- net /PC6: track 19.7 -> 13.9 mm
- net /PD7: track 14.3 -> 10.6 mm
- net /PE6: track 28.4 -> 24.9 mm
- net +5V: track 57.8 -> 54.8 mm
- net /PD4: track 13.9 -> 12.6 mm
- net /PB2: track 19.8 -> 20.9 mm
- net /PD1: track 13.5 -> 12.5 mm
- net VBUS: track 23.8 -> 24.6 mm
- net /PB4: track 20.1 -> 19.4 mm
- net /PB1: track 16.6 -> 16.8 mm, vias 1 -> 2
- net /PB6: track 11.4 -> 11.2 mm, vias 0 -> 1
- net /PB3: track 20.4 -> 20.5 mm, vias 1 -> 2
Other:
- board size 18 x 33.1 mm -> 33 x 17.8 mm
- rule trace_min: 0.15 -> 0.2
- rule via_min_size: 0.5 -> 0.6
- board text added: "PWR"
- board text added: "RST"
- board text added: "Suggested edge rail and tab locations"

Commit message: BOM complete + cleaning up traces
Parts:
- moved C6 0.60 mm to (133.2, 104.6)
- moved R3 0.20 mm to (128.3, 102.3)
- moved D2 0.20 mm to (128.3, 103.9), turned to 0 degrees
Routing:
- net GND: track 51.9 -> 47.3 mm, vias 23 -> 24
- net Net-(D2-Pad2): track 1.60 -> 2.25 mm

Commit message: add silk
Parts:
- added LOGO1: Logo_Open_Hardware_Small, josh-logos:OSHW_Logo_3.6x3.6_F.Mask, B.Cu at (140.3, 98.9)
- added SYM1: SYM_Radio_Waves_Large, josh-logos:sea-micro-silk, B.Cu at (131.9, 98.9)
- D1: value D_Schottky -> B5817WL
- U1: value ATmega32U4-MU -> ATMEGA32U4-MUR
Other:
- board text added: "5V"
- board text added: "B1"
- board text added: "B2"
- board text added: "B3"
- board text added: "B4"
- board text added: "B5"
- board text added: "B6"
- board text added: "C6"
- board text added: "D0"
- board text added: "D1"
- board text added: "D2"
- board text added: "D3"
- board text added: "D4"
- board text added: "D7"
- board text added: "E6"
- board text added: "F4"
- board text added: "F5"
- board text added: "F6"
- board text added: "F7"
- board text added: "G"
- board text added: "GND"
- board text added: "US"
- board text added: "VB"
- board text added: "nRST"
