File: hardware/0.3/pro-micro-c.sch (KiCad schematic (older format))
At the start: 22 parts, among them J1 USB_C_Receptacle_USB2.0, J2 0.1\" x 12, J3 0.1\" x 12, U1 ATmega32U4-MU, Y1 16MHz

Commit message: layout looking good
Parts:
- added SW1: KMR2, josh-buttons-switches:SW_Push_KMR2, symbol Switch:SW_Push
- D1: footprint Diode_SMD:D_SOD-123F -> josh-passives-smt:D_SOD-123F
Connections:
- net GND: now also SW1.1
- net nRST: now also SW1.2
Other:
- moved on the sheet: R4
Changed lines of the file:
@@
 L Device:R R4
 U 1 1 5E1E97C8
-P 6400 2450
-F 0 "R4" H 6470 2496 50  0000 L CNN
-F 1 "5K1" H 6470 2405 50  0000 L CNN
-F 2 "Resistor_SMD:R_0603_1608Metric" V 6330 2450 50  0001 C CNN
-F 3 "~" H 6400 2450 50  0001 C CNN
-	1    6400 2450
-	1    0    0    -1
-$EndComp
-Wire Wire Line
-	6400 2300 6400 2250
+P 6400 2200
+F 0 "R4" H 6470 2246 50  0000 L CNN
+F 1 "5K1" H 6470 2155 50  0000 L CNN
+F 2 "Resistor_SMD:R_0603_1608Metric" V 6330 2200 50  0001 C CNN
+F 3 "~" H 6400 2200 50  0001 C CNN
+	1    6400 2200
+	1    0    0    -1
+$EndComp
+Wire Wire Line
+	6400 2050 6400 2000
 $Comp
 L power:+5V #PWR014
 U 1 1 5E1F08E8
-P 6400 2250
-F 0 "#PWR014" H 6400 2100 50  0001 C CNN
-F 1 "+5V" H 6415 2423 50  0000 C CNN
-F 2 "" H 6400 2250 50  0001 C CNN
-F 3 "" H 6400 2250 50  0001 C CNN
-	1    6400 2250
+P 6400 2000
+F 0 "#PWR014" H 6400 1850 50  0001 C CNN
+F 1 "+5V" H 6415 2173 50  0000 C CNN
+F 2 "" H 6400 2000 50  0001 C CNN
+F 3 "" H 6400 2000 50  0001 C CNN
+	1    6400 2000
 	-1   0    0    -1
 $EndComp
@@
 F 0 "D1" H 2925 1734 50  0000 C CNN
 F 1 "D_Schottky" H 2925 1825 50  0000 C CNN
-F 2 "Diode_SMD:D_SOD-123F" H 2925 1950 50  0001 C CNN
+F 2 "josh-passives-smt:D_SOD-123F" H 2925 1950 50  0001 C CNN
 F 3 "~" H 2925 1950 50  0001 C CNN
 	1    2925 1950
@@
 	2025 1950 2175 1950
 Wire Wire Line
-	6400 2600 6400 2650
+	6400 2350 6400 2450
 Wire Wire Line
 	6400 2650 6900 2650
@@
 NoConn ~ 8100 5050
 NoConn ~ 8100 5150
+$Comp
+L Switch:SW_Push SW1
+U 1 1 5FD39CC7
+P 6150 2450
+F 0 "SW1" H 6150 2650 50  0000 C CNN
+F 1 "KMR2" H 6150 2350 50  0000 C CNN
+F 2 "josh-buttons-switches:SW_Push_KMR2" H 6150 2650 50  0001 C CNN
+F 3 "~" H 6150 2650 50  0001 C CNN
+	1    6150 2450
+	1    0    0    -1
+$EndComp
+Wire Wire Line
+	6350 2450 6400 2450
+Connection ~ 6400 2450
+Wire Wire Line
+	6400 2450 6400 2650
+$Comp
+L power:GND #PWR0101
+U 1 1 5FD5472A
+P 5900 2500
+F 0 "#PWR0101" H 5900 2250 50  0001 C CNN
+F 1 "GND" H 5900 2350 50  0000 C CNN
+F 2 "" H 5900 2500 50  0001 C CNN
+F 3 "" H 5900 2500 50  0001 C CNN
+	1    5900 2500
+	1    0    0    -1
+$EndComp
+Wire Wire Line
+	5900 2500 5900 2450
+Wire Wire Line
+	5900 2450 5950 2450
 $EndSCHEMATC

Commit message: BOM complete + cleaning up traces
Parts:
- C1, C2: LCSC (none) -> C1644; MPN  (none) -> CL10C150JB8NNNC; Manufacturer (none) -> Samsung Electro-Mechanics
- C3, C7, C8: LCSC (none) -> C66501; MPN  (none) -> CL10B104KO8NNNC; Manufacturer (none) -> Samsung Electro-Mechanics
- C4, C5, C6: LCSC (none) -> C1592; MPN  (none) -> CL10A105KO8NNNC; Manufacturer (none) -> Samsung Electro-Mechanics
- D1: value D_Schottky -> B5817WL; LCSC (none) -> C122853; MPN  (none) -> B5817WL; Manufacturer (none) -> Shikues
- D2: LCSC (none) -> C268294; MPN  (none) -> OSK40603C1E; Manufacturer (none) -> OptoSupply
- F1: LCSC (none) -> C210357; MPN  (none) -> MF-FSMF050X-2; Manufacturer (none) -> BOURNS
- J1: LCSC (none) -> C223907; MPN  (none) -> TYPE-C-31-M-14; Manufacturer (none) -> Korean Hroparts Elec
- J2, J3: DNP (none) -> DNP
- R1, R2, R3, R4: LCSC (none) -> C14677; MPN  (none) -> RC0603JR-075K1L; Manufacturer (none) -> YAGEO
- R5, R6: LCSC (none) -> C108405; MPN  (none) -> RC0603JR-0722RL; Manufacturer (none) -> YAGEO
- SW1: LCSC (none) -> C318893; MPN  (none) -> TS-1185EC-C-D-B; Manufacturer (none) -> XKB Connectivity
- U1: value ATmega32U4-MU -> ATMEGA32U4-MUR; LCSC (none) -> C45874; MPN  (none) -> ATMEGA32U4-MUR; Manufacturer (none) -> Microchip/Atmel
- Y1: LCSC (none) -> C164044; MPN  (none) -> TAXM16M4RDBCCT2T; Manufacturer (none) -> TAE(Zhejiang Abel Elec)
Other:
- note added: "32U4 Microcontroller"
- note added: "USB Type-C Connector / Power"
- note removed: "32u4 Microcontroller"
- note removed: "Power"
- note removed: "USB Type-C Connector"
Changed lines of the file:
@@
 encoding utf-8
 Sheet 1 1
-Title ""
-Date ""
-Rev "0"
+Title "Pro Micro C"
+Date "2020-12-11"
+Rev "0.3"
 Comp "Josh Johnson"
 Comment1 ""
@@
 P 7500 4150
 F 0 "U1" H 7050 5900 50  0000 C CNN
-F 1 "ATmega32U4-MU" V 7500 4150 50  0000 C CNN
+F 1 "ATMEGA32U4-MUR" V 7500 4150 50  0000 C CNN
 F 2 "Package_DFN_QFN:QFN-44-1EP_7x7mm_P0.5mm_EP5.2x5.2mm" H 7500 4150 50  0001 C CIN
 F 3 "http://ww1.microchip.com/downloads/en/DeviceDoc/Atmel-7766-8-bit-AVR-ATmega16U4-32U4_Datasheet.pdf" H 7500 4150 50  0001 C CNN
+F 4 "C45874" H 7500 4150 50  0001 C CNN "LCSC"
+F 5 "ATMEGA32U4-MUR" H 7500 4150 50  0001 C CNN "MPN "
+F 6 "Microchip/Atmel" H 7500 4150 50  0001 C CNN "Manufacturer"
 	1    7500 4150
 	1    0    0    -1
@@
 F 2 "josh-connectors:USB_C_TYPE-C-31-M-14" H 1350 2550 50  0001 C CNN
 F 3 "https://www.usb.org/sites/default/files/documents/usb_type-c.zip" H 1350 2550 50  0001 C CNN
+F 4 "C223907" H 1200 2550 50  0001 C CNN "LCSC"
+F 5 "TYPE-C-31-M-14" H 1200 2550 50  0001 C CNN "MPN "
+F 6 "Korean Hroparts Elec" H 1200 2550 50  0001 C CNN "Manufacturer"
 	1    1200 2550
 	1    0    0    -1
@@
 F 2 "Resistor_SMD:R_0603_1608Metric" V 2030 2150 50  0001 C CNN
 F 3 "~" H 2100 2150 50  0001 C CNN
+F 4 "C14677" H 2100 2150 50  0001 C CNN "LCSC"
+F 5 "RC0603JR-075K1L" H 2100 2150 50  0001 C CNN "MPN "
+F 6 "YAGEO" H 2100 2150 50  0001 C CNN "Manufacturer"
 	1    2100 2150
 	0    1    1    0
@@
 F 2 "Resistor_SMD:R_0603_1608Metric" V 2030 2250 50  0001 C CNN
 F 3 "~" H 2100 2250 50  0001 C CNN
+F 4 "C14677" H 2100 2250 50  0001 C CNN "LCSC"
+F 5 "RC0603JR-075K1L" H 2100 2250 50  0001 C CNN "MPN "
+F 6 "YAGEO" H 2100 2250 50  0001 C CNN "Manufacturer"
 	1    2100 2250
 	0    1    1    0
@@
 F 2 "Capacitor_SMD:C_0603_1608Metric" H 7838 1850 50  0001 C CNN
 F 3 "~" H 7800 2000 50  0001 C CNN
+F 4 "C66501" H 7800 2000 50  0001 C CNN "LCSC"
+F 5 "CL10B104KO8NNNC" H 7800 2000 50  0001 C CNN "MPN "
+F 6 "Samsung Electro-Mechanics" H 7800 2000 50  0001 C CNN "Manufacturer"
 	1    7800 2000
 	0    -1   1    0
@@
 F 2 "Capacitor_SMD:C_0603_1608Metric" H 7838 1600 50  0001 C CNN
 F 3 "~" H 7800 1750 50  0001 C CNN
+F 4 "C66501" H 7800 1750 50  0001 C CNN "LCSC"
+F 5 "CL10B104KO8NNNC" H 7800 1750 50  0001 C CNN "MPN "
+F 6 "Samsung Electro-Mechanics" H 7800 1750 50  0001 C CNN "Manufacturer"
 	1    7800 1750
 	0    -1   1    0
@@
 F 2 "Capacitor_SMD:C_0603_1608Metric" H 7838 1350 50  0001 C CNN
 F 3 "~" H 7800 1500 50  0001 C CNN
+F 4 "C1592" H 7800 1500 50  0001 C CNN "LCSC"
+F 5 "CL10A105KO8NNNC" H 7800 1500 50  0001 C CNN "MPN "
+F 6 "Samsung Electro-Mechanics" H 7800 1500 50  0001 C CNN "Manufacturer"
 	1    7800 1500
 	0    -1   1    0
@@
 F 2 "Capacitor_SMD:C_0603_1608Metric" H 5588 2600 50  0001 C CNN
 F 3 "~" H 5550 2750 50  0001 C CNN
+F 4 "C1644" H 5550 2750 50  0001 C CNN "LCSC"
+F 5 "CL10C150JB8NNNC" H 5550 2750 50  0001 C CNN "MPN "
+F 6 "Samsung Electro-Mechanics" H 5550 2750 50  0001 C CNN "Manufacturer"
 	1    5550 2750
 	0    1    1    0
@@
 F 2 "Capacitor_SMD:C_0603_1608Metric" H 5588 3000 50  0001 C CNN
 F 3 "~" H 5550 3150 50  0001 C CNN
+F 4 "C1644" H 5550 3150 50  0001 C CNN "LCSC"
+F 5 "CL10C150JB8NNNC" H 5550 3150 50  0001 C CNN "MPN "
+F 6 "Samsung Electro-Mechanics" H 5550 3150 50  0001 C CNN "Manufacturer"
 	1    5550 3150
 	0    1    1    0
@@
 F 2 "josh-oscillators:Crystal_SMD_3225-4Pin_3.2x2.5mm" H 5900 2950 50  0001 C CNN
 F 3 "~" H 5900 2950 50  0001 C CNN
+F 4 "C164044" H 5900 2950 50  0001 C CNN "LCSC"
+F 5 "TAXM16M4RDBCCT2T" H 5900 2950 50  0001 C CNN "MPN "
+F 6 "TAE(Zhejiang Abel Elec)" H 5900 2950 50  0001 C CNN "Manufacturer"
 	1    5900 2950
 	0    1    1    0
@@
 F 2 "Capacitor_SMD:C_0603_1608Metric" H 6738 4000 50  0001 C CNN
 F 3 "~" H 6700 4150 50  0001 C CNN
+F 4 "C1592" H 6700 4150 50  0001 C CNN "LCSC"
+F 5 "CL10A105KO8NNNC" H 6700 4150 50  0001 C CNN "MPN "
+F 6 "Samsung Electro-Mechanics" H 6700 4150 50  0001 C CNN "Manufacturer"
 	1    6700 4150
 	1    0    0    -1
@@
 F 2 "Capacitor_SMD:C_0603_1608Metric" H 5888 3300 50  0001 C CNN
 F 3 "~" H 5850 3450 50  0001 C CNN
+F 4 "C66501" H 5850 3450 50  0001 C CNN "LCSC"
+F 5 "CL10B104KO8NNNC" H 5850 3450 50  0001 C CNN "MPN "
+F 6 "Samsung Electro-Mechanics" H 5850 3450 50  0001 C CNN "Manufacturer"
 	1    5850 3450
 	1    0    0    -1
@@
 F 2 "Resistor_SMD:R_0603_1608Metric" V 6330 2200 50  0001 C CNN
 F 3 "~" H 6400 2200 50  0001 C CNN
+F 4 "C14677" H 6400 2200 50  0001 C CNN "LCSC"
+F 5 "RC0603JR-075K1L" H 6400 2200 50  0001 C CNN "MPN "
+F 6 "YAGEO" H 6400 2200 50  0001 C CNN "Manufacturer"
 	1    6400 2200
 	1    0    0    -1
@@
 $EndComp
 Text Notes 6750 1100 0    100  ~ 0
-32u4 Microcontroller
-Text Notes 1250 1300 0    100  ~ 0
-USB Type-C Connector
+32U4 Microcontroller
+Text Notes 1100 1300 0    100  ~ 0
+USB Type-C Connector / Power
 $Comp
 L Device:Polyfuse_Small F1
@@
 F 2 "josh-passives-smt:Fuse_0603_1608Metric" H 2325 1750 50  0001 L CNN
 F 3 "~" H 2275 1950 50  0001 C CNN
+F 4 "C210357" H 2275 1950 50  0001 C CNN "LCSC"
+F 5 "MF-FSMF050X-2" H 2275 1950 50  0001 C CNN "MPN "
+F 6 "BOURNS" H 2275 1950 50  0001 C CNN "Manufacturer"
 	1    2275 1950
 	0    1    1    0
@@
 F 2 "LED_SMD:LED_0603_1608Metric" H 3900 2450 50  0001 C CNN
 F 3 "~" H 3900 2450 50  0001 C CNN
+F 4 "C268294" H 3900 2450 50  0001 C CNN "LCSC"
+F 5 "OSK40603C1E" H 3900 2450 50  0001 C CNN "MPN "
+F 6 "OptoSupply" H 3900 2450 50  0001 C CNN "Manufacturer"
 	1    3900 2450
 	0    -1   -1   0
@@
 F 2 "Resistor_SMD:R_0603_1608Metric" V 3830 2100 50  0001 C CNN
 F 3 "~" H 3900 2100 50  0001 C CNN
+F 4 "C14677" H 3900 2100 50  0001 C CNN "LCSC"
+F 5 "RC0603JR-075K1L" H 3900 2100 50  0001 C CNN "MPN "
+F 6 "YAGEO" H 3900 2100 50  0001 C CNN "Manufacturer"
 	1    3900 2100
 	1    0    0    -1
@@
 	-1   0    0    -1
 $EndComp
-Text Notes 3700 1650 0    100  ~ 0
-Power
 $Comp
 L Device:R R5
@@
 F 2 "Resistor_SMD:R_0603_1608Metric" V 6480 3650 50  0001 C CNN
 F 3 "~" H 6550 3650 50  0001 C CNN
+F 4 "C108405" H 6550 3650 50  0001 C CNN "LCSC"
+F 5 "RC0603JR-0722RL" H 6550 3650 50  0001 C CNN "MPN "
+F 6 "YAGEO" H 6550 3650 50  0001 C CNN "Manufacturer"
 	1    6550 3650
 	0    1    1    0
@@
 F 2 "Resistor_SMD:R_0603_1608Metric" V 6480 3750 50  0001 C CNN
 F 3 "~" H 6550 3750 50  0001 C CNN
+F 4 "C108405" H 6550 3750 50  0001 C CNN "LCSC"
+F 5 "RC0603JR-0722RL" H 6550 3750 50  0001 C CNN "MPN "
+F 6 "YAGEO" H 6550 3750 50  0001 C CNN "Manufacturer"
 	1    6550 3750
 	0    1    1    0
@@
 F 2 "josh-connectors:Castellated_Short_P2.54x12" H 3000 4850 50  0001 C CNN
 F 3 "~" H 3000 4850 50  0001 C CNN
+F 4 "DNP" H 3000 4850 50  0001 C CNN "DNP"
 	1    3000 4850
 	-1   0    0    1
@@
 P 2925 1950
 F 0 "D1" H 2925 1734 50  0000 C CNN
-F 1 "D_Schottky" H 2925 1825 50  0000 C CNN
+F 1 "B5817WL" H 2925 1825 50  0000 C CNN
 F 2 "josh-passives-smt:D_SOD-123F" H 2925 1950 50  0001 C CNN
 F 3 "~" H 2925 1950 50  0001 C CNN
+F 4 "C122853" H 2925 1950 50  0001 C CNN "LCSC"
+F 5 "B5817WL" H 2925 1950 50  0001 C CNN "MPN "
+F 6 "Shikues" H 2925 1950 50  0001 C CNN "Manufacturer"
 	1    2925 1950
 	-1   0    0    1
@@
 U 1 1 5E33B6F5
 P 3500 4750
-F 0 "J3" H 3450 5500 50  0000 C CNN
-F 1 "0.1\" x 12" H 3600 5400 50  0000 C CNN
+F 0 "J3" H 3500 5500 50  0000 C CNN
+F 1 "0.1\" x 12" H 3650 5400 50  0000 C CNN
 F 2 "josh-connectors:Castellated_Short_P2.54x12" H 3500 4750 50  0001 C CNN
 F 3 "~" H 3500 4750 50  0001 C CNN
+F 4 "DNP" H 3500 4750 50  0001 C CNN "DNP"
 	1    3500 4750
 	1    0    0    -1
@@
 F 2 "Capacitor_SMD:C_0603_1608Metric" H 7188 1750 50  0001 C CNN
 F 3 "~" H 7150 1900 50  0001 C CNN
+F 4 "C1592" H 7150 1900 50  0001 C CNN "LCSC"
+F 5 "CL10A105KO8NNNC" H 7150 1900 50  0001 C CNN "MPN "
+F 6 "Samsung Electro-Mechanics" H 7150 1900 50  0001 C CNN "Manufacturer"
 	1    7150 1900
 	0    -1   1    0
@@
 F 2 "josh-buttons-switches:SW_Push_KMR2" H 6150 2650 50  0001 C CNN
 F 3 "~" H 6150 2650 50  0001 C CNN
+F 4 "C318893" H 6150 2450 50  0001 C CNN "LCSC"
+F 5 "TS-1185EC-C-D-B" H 6150 2450 50  0001 C CNN "MPN "
+F 6 "XKB Connectivity" H 6150 2450 50  0001 C CNN "Manufacturer"
 	1    6150 2450
 	1    0    0    -1

Commit message: add silk
Parts:
- added LOGO1: Logo_Open_Hardware_Small, josh-logos:OSHW_Logo_3.6x3.6_F.Mask, symbol Graphic:Logo_Open_Hardware_Small
- added SYM1: SYM_Radio_Waves_Large, josh-logos:sea-micro-silk, symbol Graphic:SYM_Radio_Waves_Large
Changed lines of the file:
@@
 PB1
 Wire Wire Line
-	8350 2650 8100 2650
-Wire Wire Line
 	8350 2750 8100 2750
 Wire Wire Line
@@
 Wire Wire Line
 	8350 4250 8100 4250
-Wire Wire Line
-	8350 4450 8100 4450
 Wire Wire Line
 	8350 4550 8100 4550
@@
 Text Label 8350 3250 2    50   ~ 0
 PB6
-NoConn ~ 8350 2650
+NoConn ~ 8100 2650
 Text Label 8350 3550 2    50   ~ 0
 PC6
@@
 Text Label 8350 4550 2    50   ~ 0
 PD7
-NoConn ~ 8350 4450
 Wire Wire Line
 	8100 4850 8350 4850
@@
 Wire Wire Line
 	5900 2450 5950 2450
+NoConn ~ 8100 4450
+$Comp
+L Graphic:Logo_Open_Hardware_Small LOGO1
+U 1 1 5FD53DBA
+P 6350 7450
+F 0 "LOGO1" H 6350 7725 50  0001 C CNN
+F 1 "Logo_Open_Hardware_Small" H 6350 7225 50  0001 C CNN
+F 2 "josh-logos:OSHW_Logo_3.6x3.6_F.Mask" H 6350 7450 50  0001 C CNN
+F 3 "~" H 6350 7450 50  0001 C CNN
+F 4 "DNP" H 6350 7450 50  0001 C CNN "DNP"
+	1    6350 7450
+	1    0    0    -1
+$EndComp
+$Comp
+L Graphic:SYM_Radio_Waves_Large SYM1
+U 1 1 5FD55A95
+P 5800 7400
+F 0 "SYM1" H 5800 7600 50  0001 C CNN
+F 1 "SYM_Radio_Waves_Large" H 5800 7150 50  0001 C CNN
+F 2 "josh-logos:sea-micro-silk" H 5800 7200 50  0001 C CNN
+F 3 "~" H 5830 7200 50  0001 C CNN
+F 4 "DNP" H 5800 7400 50  0001 C CNN "DNP"
+	1    5800 7400
+	1    0    0    -1
+$EndComp
 $EndSCHEMATC
